Commit message: Rename MERPY to MARPY (Most Affordable ROS2 Platform Yet)
Fix "Effordable" typo to "Affordable", rename all packages,
directories, files, and references from merpy to marpy.

Co-Authored-By: Claude Opus 4.6 (1M context) <noreply@anthropic.com>

File: src/marpy_description/urdf/marpy.xacro (robot description, xacro)
@@ -1,6 +1,6 @@
 <?xml version="1.0"?>
-<robot xmlns:xacro="http://www.ros.org/wiki/xacro" name="merpy">
-  <xacro:include filename="$(find merpy_description)/urdf/materials.xacro" />
-  <xacro:include filename="$(find merpy_description)/urdf/merpy_gazebo.xacro" />
+<robot xmlns:xacro="http://www.ros.org/wiki/xacro" name="marpy">
+  <xacro:include filename="$(find marpy_description)/urdf/materials.xacro" />
+  <xacro:include filename="$(find marpy_description)/urdf/marpy_gazebo.xacro" />
   <!-- ==================== Properties ==================== -->
   <!-- Wheel geometry (from CLAUDE.md specs) -->
@@ -28,5 +28,5 @@
       <origin xyz="0 0 0" rpy="0 0 0" />
       <geometry>
-        <mesh filename="package://merpy_description/meshes/base_link.STL" />
+        <mesh filename="package://marpy_description/meshes/base_link.STL" />
       </geometry>
       <material name="light_blue" />
@@ -35,5 +35,5 @@
       <origin xyz="0 0 0" rpy="0 0 0" />
       <geometry>
-        <mesh filename="package://merpy_description/meshes/base_link.STL" />
+        <mesh filename="package://marpy_description/meshes/base_link.STL" />
       </geometry>
     </collision>
@@ -52,5 +52,5 @@
       <origin xyz="0 0 0" rpy="0 0 0" />
       <geometry>
-        <mesh filename="package://merpy_description/meshes/left_wheel.STL" />
+        <mesh filename="package://marpy_description/meshes/left_wheel.STL" />
       </geometry>
       <material name="dark_grey" />
@@ -84,5 +84,5 @@
       <origin xyz="0 0 0" rpy="0 0 0" />
       <geometry>
-        <mesh filename="package://merpy_description/meshes/right_wheel.STL" />
+        <mesh filename="package://marpy_description/meshes/right_wheel.STL" />
       </geometry>
       <material name="dark_grey" />
@@ -116,5 +116,5 @@
       <origin xyz="0 0 0" rpy="0 0 0" />
       <geometry>
-        <mesh filename="package://merpy_description/meshes/caster_wheel.STL" />
+        <mesh filename="package://marpy_description/meshes/caster_wheel.STL" />
       </geometry>
       <material name="dark_grey" />

Commit message: Remove CAD STLs (moved to MakerWorld), add IMU support, and rewrite assembly docs
- Remove CAD/ folder, point all references to MakerWorld and Printables
- Add IMU link/joint to URDF from updated SolidWorks export
- Add Gazebo IMU sensor plugin (50 Hz) and gz_bridge topic
- Update meshes from new SolidWorks export
- Rewrite assembly.md with real photos, hardware tables, and step-by-step flow
- Split docs: assembly (mechanical only), wiring (electrical), firmware (flashing)
- Add assembly photos for motor mounts, caster, chassis, electronics, wheels, standoffs

Co-Authored-By: Claude Opus 4.6 (1M context) <noreply@anthropic.com>

File: src/marpy_description/urdf/marpy.xacro (robot description, xacro)
@@ -18,10 +18,10 @@
   <link name="base_link">
     <inertial>
-      <origin xyz="-0.005043 -0.0000095 0.029688" rpy="0 0 0" />
-      <mass value="0.376" />
+      <origin xyz="-0.006324 -9.655e-06 0.029104" rpy="0 0 0" />
+      <mass value="0.370" />
       <inertia
-        ixx="0.000413"  ixy="-3.78e-08" ixz="-4.35e-07"
-        iyy="0.000656"  iyz="-1.72e-08"
-        izz="0.001061" />
+        ixx="0.000410"  ixy="-3.76e-08" ixz="-5.34e-07"
+        iyy="0.000657"  iyz="-1.72e-08"
+        izz="0.001058" />
     </inertial>
     <visual>
@@ -39,4 +39,33 @@
     </collision>
   </link>
+  <!-- ==================== imu_link ==================== -->
+  <link name="imu_link">
+    <inertial>
+      <origin xyz="-0.002055 -8.047e-05 0.000508" rpy="0 0 0" />
+      <mass value="0.000548" />
+      <inertia
+        ixx="1.944e-08"  ixy="-3.334e-11" ixz="8.066e-11"
+        iyy="8.684e-09"  iyz="-4.442e-11"
+        izz="2.648e-08" />
+    </inertial>
+    <visual>
+      <origin xyz="0 0 0" rpy="0 0 0" />
+      <geometry>
+        <mesh filename="package://marpy_description/meshes/imu_link.STL" />
+      </geometry>
+      <material name="dark_grey" />
+    </visual>
+    <collision>
+      <origin xyz="0 0 0" rpy="0 0 0" />
+      <geometry>
+        <mesh filename="package://marpy_description/meshes/imu_link.STL" />
+      </geometry>
+    </collision>
+  </link>
+  <joint name="imu_joint" type="fixed">
+    <parent link="base_link" />
+    <child link="imu_link" />
+    <origin xyz="0.024 0 0.0705" rpy="0 0 0" />
+  </joint>
   <!-- ==================== left_wheel ==================== -->
   <link name="left_wheel">

File: src/marpy_description/urdf/marpy_gazebo.xacro (robot description, xacro)
@@ -59,4 +59,29 @@
     </visual>
   </gazebo>
+  <gazebo reference="imu_link">
+    <visual>
+      <material>
+        <ambient>0.2 0.2 0.2 1.0</ambient>
+        <diffuse>0.2 0.2 0.2 1.0</diffuse>
+      </material>
+    </visual>
+    <sensor name="imu_sensor" type="imu">
+      <always_on>true</always_on>
+      <update_rate>50</update_rate>
+      <topic>/imu</topic>
+      <imu>
+        <angular_velocity>
+          <x><noise type="gaussian"><mean>0</mean><stddev>0.0002</stddev></noise></x>
+          <y><noise type="gaussian"><mean>0</mean><stddev>0.0002</stddev></noise></y>
+          <z><noise type="gaussian"><mean>0</mean><stddev>0.0002</stddev></noise></z>
+        </angular_velocity>
+        <linear_acceleration>
+          <x><noise type="gaussian"><mean>0</mean><stddev>0.017</stddev></noise></x>
+          <y><noise type="gaussian"><mean>0</mean><stddev>0.017</stddev></noise></y>
+          <z><noise type="gaussian"><mean>0</mean><stddev>0.017</stddev></noise></z>
+        </linear_acceleration>
+      </imu>
+    </sensor>
+  </gazebo>
   <!--
     DiffDrive plugin: subscribes to /cmd_vel and drives the wheel joints.

Commit message: Add Printables link in BOM note and tune Gazebo physics for smoother stops
- Link ESP32-CAM GoPro case in BOM note
- Reduce contact stiffness, increase contact/joint damping
- Add deceleration limits to diff drive plugin

Co-Authored-By: Claude Opus 4.6 (1M context) <noreply@anthropic.com>

File: src/marpy_description/urdf/marpy.xacro (robot description, xacro)
@@ -98,5 +98,5 @@
     <axis xyz="0 1 0" />
     <limit effort="10" velocity="10" />
-    <dynamics damping="0.1" friction="0.1" />
+    <dynamics damping="0.5" friction="0.3" />
   </joint>
   <!-- ==================== right_wheel ==================== -->
@@ -130,5 +130,5 @@
     <axis xyz="0 1 0" />
     <limit effort="10" velocity="10" />
-    <dynamics damping="0.1" friction="0.1" />
+    <dynamics damping="0.5" friction="0.3" />
   </joint>
   <!-- ==================== caster_wheel ==================== -->

File: src/marpy_description/urdf/marpy_gazebo.xacro (robot description, xacro)
@@ -5,6 +5,6 @@
     <mu1>1.0</mu1>
     <mu2>0.5</mu2>
-    <kp>1e6</kp>
-    <kd>100.0</kd>
+    <kp>1e5</kp>
+    <kd>1e3</kd>
     <minDepth>0.001</minDepth>
     <maxVel>1.0</maxVel>
@@ -13,6 +13,6 @@
     <mu1>1.0</mu1>
     <mu2>0.5</mu2>
-    <kp>1e6</kp>
-    <kd>100.0</kd>
+    <kp>1e5</kp>
+    <kd>1e3</kd>
     <minDepth>0.001</minDepth>
     <maxVel>1.0</maxVel>
@@ -22,6 +22,6 @@
     <mu1>0.01</mu1>
     <mu2>0.01</mu2>
-    <kp>1e6</kp>
-    <kd>100.0</kd>
+    <kp>1e5</kp>
+    <kd>1e3</kd>
     <minDepth>0.001</minDepth>
   </gazebo>
@@ -97,5 +97,7 @@
       <wheel_radius>0.033</wheel_radius>
       <max_linear_acceleration>1.0</max_linear_acceleration>
+      <max_linear_deceleration>1.5</max_linear_deceleration>
       <max_angular_acceleration>2.0</max_angular_acceleration>
+      <max_angular_deceleration>3.0</max_angular_deceleration>
       <topic>/cmd_vel</topic>
     </plugin>
